Commit message: small configuration changes

File: mir_robots/mir_hardware_config/youbot-brsu-2/urdf/robot.urdf.xacro (robot description, xacro)
@@ -55,5 +55,5 @@
      <!-- camera calibration -->
       <!-- <origin xyz="0.035 0.020 0.0" rpy="0.0 1.22 0.0" /> -->
-      <origin xyz="0.010 -0.005 0.0" rpy="0.0 1.22 0.0" />
+      <origin xyz="-0.030 0.015 0.0" rpy="0.0 1.22 0.0" />
   </xacro:sensor_d435>
   <!-- tower middle camera -->

Commit message: GO24 - day 2 changes

File: mir_robots/mir_hardware_config/youbot-brsu-2/urdf/robot.urdf.xacro (robot description, xacro)
@@ -55,5 +55,5 @@
      <!-- camera calibration -->
       <!-- <origin xyz="0.035 0.020 0.0" rpy="0.0 1.22 0.0" /> -->
-      <origin xyz="-0.030 0.015 0.0" rpy="0.0 1.22 0.0" />
+      <origin xyz="-0.026 0.020 0.0" rpy="0.0 1.22 0.0" />
   </xacro:sensor_d435>
   <!-- tower middle camera -->

Commit message: GO24 - day 3 - pre ATT1

File: mir_robots/mir_hardware_config/youbot-brsu-2/urdf/robot.urdf.xacro (robot description, xacro)
@@ -55,5 +55,5 @@
      <!-- camera calibration -->
       <!-- <origin xyz="0.035 0.020 0.0" rpy="0.0 1.22 0.0" /> -->
-      <origin xyz="-0.026 0.020 0.0" rpy="0.0 1.22 0.0" />
+      <origin xyz="-0.026 0.005 0.0" rpy="0.0 1.22 0.0" />
   </xacro:sensor_d435>
   <!-- tower middle camera -->
